File: CAD/CANUSB4/CANUSB4.kicad_pcb (KiCad board)
At the start: 2 copper layers, 80 x 67.5 mm, 50 parts, among them J1 CAN, J2 USB_B, J3 ISP, J4 ISP, SW1 PB, U1 LM7805CT, U2 MCP2562-E-P, U3 ADUM4160, U4 PIC18F26K80, U5 PIC18F14K50, Y1 12MHz, Y2 4MHz

Commit message: Add pdf files, CAD files
Parts:
- removed the REF** at (16.3, -3.30)
- added C4: 100nF, Capacitor_SMD:C_1206_3216Metric_Pad1.33x1.80mm_HandSolder, F.Cu at (59.2, -13.0)
- added C7: 100nF, Capacitor_SMD:C_1206_3216Metric_Pad1.33x1.80mm_HandSolder, F.Cu at (52.6, -21.3)
- added C8: 100nF, Capacitor_SMD:C_1206_3216Metric_Pad1.33x1.80mm_HandSolder, F.Cu at (38.8, -11.7)
- added JP3: D+, Connector_PinSocket_2.54mm:PinSocket_1x02_P2.54mm_Vertical, F.Cu at (24.1, -14.0)
- added JP4: D-, Connector_PinSocket_2.54mm:PinSocket_1x02_P2.54mm_Vertical, F.Cu at (27.9, -14.0)
- added R7: 27R, Resistor_SMD:R_1206_3216Metric, F.Cu at (19.4, -11.4)
- added R8: 27R, Resistor_SMD:R_1206_3216Metric, F.Cu at (19.4, -14.0)
- added REF**: KiCad-Logo2_5mm_SilkScreen, Symbol:KiCad-Logo2_5mm_SilkScreen, F.Cu at (16.8, -3.56)
- D1: footprint PCM_Diode_THT_AKL:D_DO-41_SOD81_P7.62mm_Horizontal -> Diode_THT:D_DO-41_SOD81_P10.16mm_Horizontal
- JP1, JP2: footprint Connector_PinSocket_1.27mm:PinSocket_1x02_P1.27mm_Vertical -> Connector_PinSocket_2.54mm:PinSocket_1x02_P2.54mm_Vertical
- JP5: renamed from JP3; footprint Connector_PinSocket_1.27mm:PinSocket_1x02_P1.27mm_Vertical -> Connector_PinSocket_2.54mm:PinSocket_1x02_P2.54mm_Vertical
- R1, R2: value 24R -> 27R
- U1: value LM7805CT -> 78M05
- moved REF** 19.6 mm to (65.5, -3.05)
- moved D1 1.93 mm to (67.9, -38.0)
- moved JP1 1.80 mm to (59.4, -58.9)
- moved U1 1.33 mm to (61.5, -32.6)
- moved R1 1.03 mm to (59.2, -10.4)
- moved R11 0.78 mm to (38.8, -14.2)
- moved C5 0.25 mm to (53.0, -25.7)
- renumbered C7 to C10, C8 to C11, C9 to C12, C10 to C13, C11 to C14, C12 to C15, C13 to C16, C4 to C5, C5 to C6, C6 to C9, R8 to R10, R9 to R11, R10 to R12, R11 to R13, R7 to R9
Connections:
- J3 pad 4: /DD+ -> Net-(J3-PGD/ICSPDAT)
- J3 pad 5: /DD- -> Net-(J3-PGC/ICSPCLK)
- U3 pad 10: /DD+ -> Net-(U3-DD+)
- U3 pad 11: /DD- -> Net-(U3-DD-)
- U5 pad 18: /DD- -> Net-(J3-PGC/ICSPCLK)
- U5 pad 19: /DD+ -> Net-(J3-PGD/ICSPDAT)
Routing:
- net Net-(U3-DD-): track 0.00 -> 48.0 mm, vias 0 -> 2
- net GND: track 353.4 -> 311.3 mm, vias 3 -> 1
- net Net-(U3-DD+): track 0.00 -> 40.9 mm, vias 0 -> 2
- net Net-(J3-PGD/ICSPDAT): track 0.00 -> 22.4 mm
- net /DD+: track 25.6 -> 3.30 mm
- net /DD-: track 34.2 -> 16.0 mm, vias 0 -> 1
- net GNDA: track 153.2 -> 169.0 mm, vias 0 -> 1
- net Net-(J3-PGC/ICSPCLK): track 0.00 -> 13.5 mm
- net Net-(U3-PIN): track 2.54 -> 15.2 mm
- net +5V: track 228.9 -> 236.3 mm, vias 4 -> 5
- net Net-(U3-PDEN): track 2.54 -> 6.51 mm
- net +5VA: track 171.6 -> 167.8 mm
- net Net-(U3-UD+): track 11.9 -> 13.8 mm
- net /CANH: track 21.3 -> 19.7 mm
- net Net-(J4-PGD/ICSPDAT): track 91.8 -> 93.0 mm
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Other:
- board text added: "CANUSB4-ISO 04-2026-1.01 DL7BJ"
- board text removed: "CANUSB4-ISO 01-2026-1.00 DL7BJ"
