File: CAD/CANUSB4/CANUSB4.kicad_sch (KiCad schematic)
At the start: 48 parts, among them J1 CAN, J2 USB_B, J3 ISP, J4 ISP, SW1 PB, U1 LM7805CT, U2 MCP2562-E-P, U3 ADUM4160, U4 PIC18F26K80, U5 PIC18F14K50, Y1 12MHz, Y2 4MHz

Commit message: Add pdf files, CAD files
Parts:
- removed D1: 1N5819, PCM_Diode_THT_AKL:D_DO-41_SOD81_P7.62mm_Horizontal, symbol PCM_Diode_Schottky_AKL:1N5819
- removed U1: LM7805CT, Package_TO_SOT_SMD:TO-252-3_TabPin2, symbol PCM_Voltage_Regulator_AKL:LM7805CT
- added C4, C7, C8: 100nF, Capacitor_SMD:C_1206_3216Metric_Pad1.33x1.80mm_HandSolder, symbol Device:C_Small
- added D1: 1N5819, Diode_THT:D_DO-41_SOD81_P10.16mm_Horizontal, symbol Diode:1N5819
- added JP3: D+, Connector_PinSocket_2.54mm:PinSocket_1x02_P2.54mm_Vertical, symbol Jumper:Jumper_2_Bridged
- added JP4: D-, Connector_PinSocket_2.54mm:PinSocket_1x02_P2.54mm_Vertical, symbol Jumper:Jumper_2_Bridged
- added R7, R8: 27R, Resistor_SMD:R_1206_3216Metric, symbol Device:R_Small
- added U1: 78M05, Package_TO_SOT_SMD:TO-252-3_TabPin2, symbol Regulator_Linear:KA78M05_TO252
- JP1, JP2: footprint Connector_PinSocket_1.27mm:PinSocket_1x02_P1.27mm_Vertical -> Connector_PinSocket_2.54mm:PinSocket_1x02_P2.54mm_Vertical
- JP5: renamed from JP3; footprint Connector_PinSocket_1.27mm:PinSocket_1x02_P1.27mm_Vertical -> Connector_PinSocket_2.54mm:PinSocket_1x02_P2.54mm_Vertical
- R1, R2: value 24R -> 27R
- renumbered C7 to C10, C8 to C11, C9 to C12, C10 to C13, C11 to C14, C12 to C15, C13 to C16, C4 to C5, C5 to C6, C6 to C9, R8 to R10, R9 to R11, R10 to R12, R11 to R13, R7 to R9
Connections:
- net +12V: now also D1.2 (A)
- net +5V: now also C8.1, U1.3 (VO)
- net DD+: now also JP3.2 (B), R7.1; no longer J3.4 (PGD/ICSPDAT), U3.10 (DD+), U5.19 (RA0/IOCA0/D+/PGD)
- net DD-: now also JP4.2 (B), R8.2; no longer J3.5 (PGC/ICSPCLK), U3.11 (DD-), U5.18 (RA1/IOCA1/D-/PGC)
- net GND: now also C7.2, C8.2, U1.2 (GND)
- net GNDA: now also C4.2
- net at C2.1, C3.1: now also D1.1 (K), U1.1 (VI)
- net at U3.12 (PIN), U3.13 (SPD), U3.14 (VDD2): now also C7.1
- net at U3.3 (VDD1), U3.4 (PDEN), U3.5 (SPU): now also C4.1
- new net: J3.4 (PGD/ICSPDAT), JP3.1 (A), U5.19 (RA0/IOCA0/D+/PGD)
- new net: J3.5 (PGC/ICSPCLK), JP4.1 (A), U5.18 (RA1/IOCA1/D-/PGC)
- new net: R8.1, U3.11 (DD-)
- new net: R7.2, U3.10 (DD+)
Other:
- title: CANUSB4 -> CANUSB4-ISO
